Commit message: Remove duplicate pi definition and fix flake8

File: src/ur5_robot_description/urdf/ur5_robot.urdf.xacro (robot description, xacro)
@@ -2,5 +2,4 @@
 <robot xmlns:xacro="http://www.ros.org/wiki/xacro" name="ur5">
   <!-- Common properties -->
-  <xacro:property name="pi" value="3.14159265359" />
   <!-- UR5 specific properties -->
   <xacro:property name="shoulder_height" value="0.089159" />
